Commit message: Gripper works

File: src/DOBOT_6Axis_ROS2_V3/gripper_pgc_description/urdf/gripper_pgc.xacro (robot description, xacro)
@@ -70,4 +70,6 @@
   </inertial>
 </link>
+<link name="gripper_middle">
+</link>
 <joint name="left_joint" type="prismatic">
   <origin xyz="-0.01085 0.0 0.0793" rpy="0 0 0"/>
@@ -75,6 +77,5 @@
   <child link="left_1"/>
   <axis xyz="0.0 1.0 0.0"/>
-  <limit upper="0.0" lower="0.0" effort="100" velocity="100"/>
-  <mimic joint="right_joint" multiplier="-1"/>
+  <limit upper="0.013" lower="0.0" effort="20" velocity="0.2"/>
 </joint>
 <joint name="right_joint" type="prismatic">
@@ -82,6 +83,7 @@
   <parent link="gripper_base_link"/>
   <child link="right_1"/>
-  <axis xyz="0.0 1.0 0.0"/>
-  <limit upper="-0.013" lower="0.000" effort="100" velocity="100"/>
+  <axis xyz="0.0 -1.0 0.0"/>
+  <limit upper="0.013" lower="0.000" effort="20" velocity="0.2"/>
+    <mimic joint="left_joint" multiplier="1"/>
 </joint>
 <joint name="Rigid 10" type="fixed">
@@ -90,3 +92,8 @@
   <child link="stylus_frame_1"/>
 </joint>
+<joint name="gripper_middle_joint" type="fixed">
+  <origin xyz="-0.025 0 0.19" rpy="0 -0.523599 0"/>
+  <parent link="gripper_base_link"/>
+  <child link="gripper_middle"/>
+</joint>
 </robot>

File: src/DOBOT_6Axis_ROS2_V3/nova2_with_gripper_moveit_config/config/nova2_with_gripper.ros2_control.xacro (robot description, xacro)
@@ -50,8 +50,8 @@
                 <state_interface name="velocity"/>
             </joint>
-            <joint name="right_joint">
+            <joint name="left_joint">
                 <command_interface name="position"/>
                 <state_interface name="position">
-                  <param name="initial_value">${initial_positions['right_joint']}</param>
+                  <param name="initial_value">${initial_positions['left_joint']}</param>
                 </state_interface>
                 <state_interface name="velocity"/>
